Commit message: fix base and not use gripper

File: doosan-robot/dsr_description/xacro/base_m0609.urdf.xacro (robot description, xacro)
@@ -2,5 +2,5 @@
 <robot xmlns:xacro="http://www.ros.org/wiki/xacro" name="m0609" >
   <xacro:arg name="color"   default="white"/>
-  <xacro:arg name="gripper" default="robotiq_2f"/>
+  <xacro:arg name="gripper" default="none"/>
   <xacro:property name="cr" value="$(arg color)"/>
   <xacro:property name="gr" value="$(arg gripper)"/>
@@ -14,10 +14,10 @@
   <xacro:m0609 namespace="$(arg namespace)"/>
   <link name="world" />
-  <!-- <xacro:if value="${gr == 'robotiq_2f'}"> -->
+  <xacro:if value="${gr == 'robotiq_2f'}">
      <xacro:include filename="$(find dsr_description)/xacro/robotiq_2f.urdf.xacro" />
-  <!-- </xacro:if> -->
+  </xacro:if>
   <!-- World fixed joint-->
   <joint name="world_fixed" type="fixed">
-    <origin xyz="0 0 0" rpy="0 0 0"/>
+    <origin xyz="0 0 0.05" rpy="0 0 0"/>
     <parent link="world"/>
     <child link="mobile_base"/>
@@ -51,5 +51,5 @@
 		  <child link="base_0"/>
         <origin
-      xyz="-0.15008 -0.0048392 0.81535"
+      xyz="-0.15008 -0.0048392 0.800"
       rpy="0 0 0" />
     <axis

File: doosan-robot/moveit_config_base_m0609/config/gazebo_m0609.urdf (robot description, URDF)
Before this commit: robot m0609, 21 links, 20 joints
Links:
- removed link robotiq_85_base_link
- removed link robotiq_85_left_finger_link
- removed link robotiq_85_left_finger_tip_link
- removed link robotiq_85_left_inner_knuckle_link
- removed link robotiq_85_left_knuckle_link
- removed link robotiq_85_right_finger_link
- removed link robotiq_85_right_finger_tip_link
- removed link robotiq_85_right_inner_knuckle_link
- removed link robotiq_85_right_knuckle_link
- removed link robotiq_coupler
Joints:
- removed joint robotiq_85_base_joint
- removed joint robotiq_85_left_finger_joint
- removed joint robotiq_85_left_finger_tip_joint
- removed joint robotiq_85_left_inner_knuckle_joint
- removed joint robotiq_85_left_knuckle_joint
- removed joint robotiq_85_right_finger_joint
- removed joint robotiq_85_right_finger_tip_joint
- removed joint robotiq_85_right_inner_knuckle_joint
- removed joint robotiq_85_right_knuckle_joint
- removed joint robotiq_coupler_joint
- joint fixed: origin xyz=-0.15008 -0.0048392 0.81535 rpy=0 0 0 -> xyz=-0.15008 -0.0048392 0.800 rpy=0 0 0
- joint world_fixed: origin xyz=0 0 0 rpy=0 0 0 -> xyz=0 0 0.05 rpy=0 0 0
